Commit message: :recycle: 파일 및 폴더 정리 && 데이터 수집 로직 수정

File: custom_panda_description/urdf/panda_with_robotiq.urdf (robot description, URDF)
Before this commit: robot panda_with_robotiq, 19 links, 18 joints
Links:
- added link gripper_tip_link, mass 0.001; collision box size=0.01 0.01 0.01; visual box size=0.01 0.01 0.01
Joints:
- added joint gripper_tip_joint: type fixed, parent robotiq_85_base_link, child gripper_tip_link, origin xyz=0 0 0.25 rpy=0 0 0

Commit message: 6D invert 수정

File: custom_panda_description/urdf/panda_with_robotiq.urdf (robot description, URDF)
Before this commit: robot panda_with_robotiq, 20 links, 19 joints
Joints:
- joint gripper_tip_joint: origin xyz=0 0 0.25 rpy=0 0 0 -> xyz=0 0 0.20 rpy=0 0 0
- joint panda_to_gripper: origin xyz=0 0 0 rpy=0 0 -0.785398163397 -> xyz=0 0 0 rpy=0 0 -2.35619449019

Commit message: scale 조절

File: custom_panda_description/urdf/panda_with_robotiq.urdf (robot description, URDF)
Before this commit: robot panda_with_robotiq, 20 links, 19 joints
Joints:
- joint panda_to_gripper: origin xyz=0 0 0 rpy=0 0 -2.35619449019 -> xyz=0 0 0 rpy=0 0 0.785398163397

Commit message: URDF joint-4 수정

File: custom_panda_description/urdf/panda_with_robotiq.urdf (robot description, URDF)
Before this commit: robot panda_with_robotiq, 20 links, 19 joints
Joints:
- joint panda_joint4: limit lower=-3.1416 upper=0.0873 effort=87 velocity=2.3925 -> lower=-3.0718 upper=-0.0698 effort=87 velocity=2.3925
